File: lipo-protection.sch (KiCad schematic (older format))
At the start: 10 parts, among them P1 P-, P2 B-, P3 B+, P4 P+, Q1 Q_NMOS_GSD, Q2 Q_NMOS_GSD, U1 S-8200A

Commit message: start layout
Parts:
- removed P1: P-, kicadlib:TEST_0.100, symbol TST
- removed P2: B-, kicadlib:TEST_0.100, symbol TST
- removed P3: B+, kicadlib:TEST_0.100, symbol TST
- removed P4: P+, kicadlib:TEST_0.100, symbol TST
- added J1, J2: 2_PIN_HDR, kicadlib:TH_JST_2PIN_RIGHTANGLE, symbol 2_PIN_HDR
- Q1, Q2: footprint (none) -> kicadlib:SMD_SOT23-3
Connections:
- net GND: now also J1.2
- net batt+: now also J1.1, J2.1
- net power-: now reaches Q2.2 (S), R1.2
- net power-: now also J2.2
Other:
- note added: "Battery connector"
- note added: "Power out"
Changed lines of the file:
@@
 LIBS:valves
 LIBS:kicadlib
+LIBS:lipo-protection-cache
 EELAYER 25 0
 EELAYER END
@@
 $EndComp
 $Comp
-L TST P3
-U 1 1 573738BD
-P 6650 3600
-F 0 "P3" H 6650 3900 50  0000 C BNN
-F 1 "B+" H 6650 3850 50  0000 C CNN
-F 2 "kicadlib:TEST_0.100" H 6650 3600 60  0001 C CNN
-F 3 "" H 6650 3600 60  0000 C CNN
-	1    6650 3600
-	1    0    0    -1
-$EndComp
-$Comp
-L TST P2
-U 1 1 57373A00
-P 6100 3200
-F 0 "P2" H 6100 3500 50  0000 C BNN
-F 1 "B-" H 6100 3450 50  0000 C CNN
-F 2 "kicadlib:TEST_0.100" H 6100 3200 60  0001 C CNN
-F 3 "" H 6100 3200 60  0000 C CNN
-	1    6100 3200
-	1    0    0    -1
-$EndComp
-$Comp
 L C C1
 U 1 1 57373A37
@@
 $EndComp
 Wire Wire Line
-	6100 3200 6100 3300
-Wire Wire Line
 	6100 3250 6000 3250
 Wire Wire Line
@@
 Wire Wire Line
 	6000 3450 5900 3450
-Connection ~ 6100 3250
-$Comp
-L TST P4
-U 1 1 57374297
-P 6850 3600
-F 0 "P4" H 6850 3900 50  0000 C BNN
-F 1 "P+" H 6850 3850 50  0000 C CNN
-F 2 "kicadlib:TEST_0.100" H 6850 3600 60  0001 C CNN
-F 3 "" H 6850 3600 60  0000 C CNN
-	1    6850 3600
-	1    0    0    -1
-$EndComp
-Connection ~ 6650 3600
 $Comp
 L GND #PWR02
@@
 Wire Wire Line
 	6550 4100 6550 4000
-$Comp
-L TST P1
-U 1 1 57374408
-P 4600 3500
-F 0 "P1" H 4600 3800 50  0000 C BNN
-F 1 "P-" H 4600 3750 50  0000 C CNN
-F 2 "kicadlib:TEST_0.100" H 4600 3500 60  0001 C CNN
-F 3 "" H 4600 3500 60  0000 C CNN
-	1    4600 3500
-	1    0    0    -1
-$EndComp
 NoConn ~ 5900 3750
 Wire Wire Line
@@
 F 0 "Q2" H 4400 3800 50  0000 R CNN
 F 1 "Q_NMOS_GSD" H 4750 3700 50  0000 R CNN
-F 2 "" H 4300 3850 29  0001 C CNN
+F 2 "kicadlib:SMD_SOT23-3" H 4300 3850 29  0001 C CNN
 F 3 "" H 4100 3750 60  0000 C CNN
 	1    4100 3750
@@
 F 0 "Q1" H 4400 3300 50  0000 R CNN
 F 1 "Q_NMOS_GSD" H 4750 3200 50  0000 R CNN
-F 2 "" H 4300 3350 29  0001 C CNN
+F 2 "kicadlib:SMD_SOT23-3" H 4300 3350 29  0001 C CNN
 F 3 "" H 4100 3250 60  0000 C CNN
 	1    4100 3250
@@
 Wire Wire Line
 	4800 3450 5100 3450
+Wire Wire Line
+	6100 3250 6100 3300
+Text Label 4600 3500 2    60   ~ 0
+power-
+$Comp
+L 2_PIN_HDR J1
+U 1 1 573753C0
+P 4400 2550
+F 0 "J1" H 4400 2400 60  0000 C CNN
+F 1 "2_PIN_HDR" H 4400 2850 60  0000 C CNN
+F 2 "kicadlib:TH_JST_2PIN_RIGHTANGLE" H 4400 2550 60  0001 C CNN
+F 3 "" H 4400 2550 60  0000 C CNN
+	1    4400 2550
+	1    0    0    -1
+$EndComp
+$Comp
+L 2_PIN_HDR J2
+U 1 1 573754DE
+P 6200 2550
+F 0 "J2" H 6200 2400 60  0000 C CNN
+F 1 "2_PIN_HDR" H 6200 2850 60  0000 C CNN
+F 2 "kicadlib:TH_JST_2PIN_RIGHTANGLE" H 6200 2550 60  0001 C CNN
+F 3 "" H 6200 2550 60  0000 C CNN
+	1    6200 2550
+	-1   0    0    -1
+$EndComp
+Text Label 5900 2400 2    60   ~ 0
+batt+
+Wire Wire Line
+	5900 2400 6000 2400
+Text Label 4700 2400 0    60   ~ 0
+batt+
+Wire Wire Line
+	4600 2400 4700 2400
+Text Label 4700 2550 0    60   ~ 0
+batt-
+Wire Wire Line
+	4700 2550 4600 2550
+Text Label 5900 2550 2    60   ~ 0
+power-
+Wire Wire Line
+	5900 2550 6000 2550
+Text Notes 6000 2050 0    60   ~ 0
+Power out
+Text Notes 4250 2050 0    60   ~ 0
+Battery connector
 $EndSCHEMATC
