File: lipo-protection.kicad_pcb (KiCad board)
At the start: 2 copper layers, 23.5 x 8.3 mm, 8 parts, among them J1 2_PIN_HDR, J2 2_PIN_HDR, Q1 Q_NMOS_GSD, Q2 Q_NMOS_GSD, U1 S-8200A

Commit message: finish layout
Routing:
- net /batt+: track 0.00 -> 20.3 mm
- net /power-: track 0.00 -> 10.7 mm
- net Net-(R2-Pad2): track 0.00 -> 5.78 mm, vias 0 -> 2
- net Net-(Q2-Pad1): track 0.00 -> 5.25 mm
- net GND: track 0.00 -> 3.85 mm
- net Net-(Q1-Pad3): track 0.00 -> 3.81 mm
- net Net-(R1-Pad1): track 0.00 -> 3.74 mm
- net Net-(Q1-Pad1): track 0.00 -> 2.84 mm
- added copper zone on B.Cu, net GND
- added copper zone on F.Cu, net GND
Other:
- outline, holes or cut-outs redrawn
- board text added: "github.com/noahp/ lipo-protection v0"
Changed lines of the file:
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@@
   (general
     (links 13)
-    (no_connects 13)
-    (area 116.764999 65.874999 140.425001 74.375001)
+    (no_connects 0)
+    (area 116.774999 65.874999 140.425001 74.375001)
     (thickness 1.6)
-    (drawings 4)
-    (tracks 0)
+    (drawings 9)
+    (tracks 47)
     (zones 0)
     (modules 8)
@@
     (last_trace_width 0.25)
     (trace_clearance 0.2)
-    (zone_clearance 0.508)
+    (zone_clearance 0.254)
     (zone_45_only no)
     (trace_min 0.2)
@@
     )
   )
-  (gr_line (start 116.85 74.3) (end 140.35 74.3) (angle 90) (layer Edge.Cuts) (width 0.15))
-  (gr_line (start 116.85 74.3) (end 116.85 65.95) (angle 90) (layer Edge.Cuts) (width 0.15))
-  (gr_line (start 140.35 65.95) (end 140.35 74.3) (angle 90) (layer Edge.Cuts) (width 0.15))
-  (gr_line (start 140.35 65.95) (end 116.85 65.95) (angle 90) (layer Edge.Cuts) (width 0.15))
+  (gr_text "github.com/noahp/\nlipo-protection\nv0" (at 128.35 68.4) (layer B.Mask)
+    (effects (font (size 0.75 0.75) (thickness 0.12)) (justify mirror))
+  )
+  (gr_line (start 116.85 73.55) (end 116.85 66.7) (angle 90) (layer Edge.Cuts) (width 0.15))
+  (gr_line (start 139.6 74.3) (end 117.6 74.3) (angle 90) (layer Edge.Cuts) (width 0.15))
+  (gr_line (start 140.35 66.7) (end 140.35 73.55) (angle 90) (layer Edge.Cuts) (width 0.15))
+  (gr_line (start 117.6 65.95) (end 139.6 65.95) (angle 90) (layer Edge.Cuts) (width 0.15))
+  (gr_line (start 140.35 66.7) (end 139.6 65.95) (angle 90) (layer Edge.Cuts) (width 0.15))
+  (gr_line (start 139.6 74.3) (end 140.35 73.55) (angle 90) (layer Edge.Cuts) (width 0.15))
+  (gr_line (start 116.85 73.55) (end 117.6 74.3) (angle 90) (layer Edge.Cuts) (width 0.15))
+  (gr_line (start 117.6 65.95) (end 116.85 66.7) (angle 90) (layer Edge.Cuts) (width 0.15))
+  (segment (start 132.461 67.31) (end 132.461 67.11) (width 0.25) (layer F.Cu) (net 1))
+  (segment (start 132.461 67.11) (end 131.885999 66.534999) (width 0.25) (layer F.Cu) (net 1))
+  (segment (start 131.885999 66.534999) (end 129.861001 66.534999) (width 0.25) (layer F.Cu) (net 1))
+  (segment (start 129.861001 66.534999) (end 129.286 67.11) (width 0.25) (layer F.Cu) (net 1))
+  (segment (start 129.286 67.11) (end 129.286 67.31) (width 0.25) (layer F.Cu) (net 1))
+  (segment (start 132.461 67.51) (end 132.461 67.31) (width 0.25) (layer F.Cu) (net 1))
+  (segment (start 132.461 67.31) (end 132.461 68.056) (width 0.25) (layer F.Cu) (net 1))
+  (segment (start 132.461 68.056) (end 135.525 71.12) (width 0.25) (layer F.Cu) (net 1))
+  (segment (start 135.525 71.12) (end 136.525 71.12) (width 0.25) (layer F.Cu) (net 1))
+  (segment (start 120.65 69.215) (end 121.65 69.215) (width 0.25) (layer F.Cu) (net 1))
+  (segment (start 121.65 69.215) (end 124.255 66.61) (width 0.25) (layer F.Cu) (net 1))
+  (segment (start 124.255 66.61) (end 128.086 66.61) (width 0.25) (layer F.Cu) (net 1))
+  (segment (start 128.086 66.61) (end 128.786 67.31) (width 0.25) (layer F.Cu) (net 1))
+  (segment (start 128.786 67.31) (end 129.286 67.31) (width 0.25) (layer F.Cu) (net 1))
+  (segment (start 131.318999 72.068999) (end 131.5 72.25) (width 0.25) (layer F.Cu) (net 2))
+  (segment (start 132.294 69.408) (end 131.394 69.408) (width 0.25) (layer F.Cu) (net 2))
+  (segment (start 131.318999 69.483001) (end 131.318999 72.068999) (width 0.25) (layer F.Cu) (net 2))
+  (segment (start 131.394 69.408) (end 131.318999 69.483001) (width 0.25) (layer F.Cu) (net 2))
+  (segment (start 130.429 73.025) (end 130.429 72.325) (width 0.25) (layer F.Cu) (net 3))
+  (segment (start 130.429 72.325) (end 130.769001 71.984999) (width 0.25) (layer F.Cu) (net 3))
+  (segment (start 130.769001 71.984999) (end 130.769001 70.433001) (width 0.25) (layer F.Cu) (net 3))
+  (segment (start 130.769001 70.433001) (end 130.694 70.358) (width 0.25) (layer F.Cu) (net 3))
+  (segment (start 130.694 70.358) (end 129.794 70.358) (width 0.25) (layer F.Cu) (net 3))
+  (segment (start 135 67.35) (end 134.025 67.35) (width 0.25) (layer F.Cu) (net 4))
+  (segment (start 134.025 67.35) (end 133.985 67.31) (width 0.25) (layer F.Cu) (net 4))
+  (segment (start 133.536551 70.015449) (end 133.536551 68.813449) (width 0.25) (layer B.Cu) (net 4))
+  (via (at 135 67.35) (size 0.6) (drill 0.4) (layers F.Cu B.Cu) (net 4))
+  (segment (start 133.536551 68.813449) (end 135 67.35) (width 0.25) (layer B.Cu) (net 4))
+  (segment (start 133.194 70.358) (end 133.536551 70.015449) (width 0.25) (layer F.Cu) (net 4))
+  (segment (start 133.6 69.952) (end 133.536551 70.015449) (width 0.25) (layer F.Cu) (net 4))
+  (via (at 133.536551 70.015449) (size 0.6) (drill 0.4) (layers F.Cu B.Cu) (net 4))
+  (segment (start 132.294 70.358) (end 133.194 70.358) (width 0.25) (layer F.Cu) (net 4))
+  (segment (start 127 69.53) (end 129.672 69.53) (width 0.25) (layer F.Cu) (net 5))
+  (segment (start 129.672 69.53) (end 129.794 69.408) (width 0.25) (layer F.Cu) (net 5))
+  (segment (start 129.794 71.308) (end 129.794 73.421002) (width 0.25) (layer F.Cu) (net 6))
+  (segment (start 129.794 73.421002) (end 129.415001 73.800001) (width 0.25) (layer F.Cu) (net 6))
+  (segment (start 129.415001 73.800001) (end 128.360001 73.800001) (width 0.25) (layer F.Cu) (net 6))
+  (segment (start 128.360001 73.800001) (end 127.9 73.34) (width 0.25) (layer F.Cu) (net 6))
+  (segment (start 127.9 73.34) (end 127 73.34) (width 0.25) (layer F.Cu) (net 6))
+  (segment (start 124.5 72.39) (end 124.5 68.58) (width 0.25) (layer F.Cu) (net 8))
+  (segment (start 122.425001 72.990001) (end 125.449999 72.990001) (width 0.25) (layer F.Cu) (net 9))
+  (segment (start 125.449999 72.990001) (end 127 71.44) (width 0.25) (layer F.Cu) (net 9))
+  (segment (start 120.65 71.215) (end 122.425001 72.990001) (width 0.25) (layer F.Cu) (net 9))
+  (segment (start 128.905 73.025) (end 128.905 72.325) (width 0.25) (layer F.Cu) (net 9))
+  (segment (start 128.905 72.325) (end 128.02 71.44) (width 0.25) (layer F.Cu) (net 9))
+  (segment (start 128.02 71.44) (end 127.9 71.44) (width 0.25) (layer F.Cu) (net 9))
+  (segment (start 127.9 71.44) (end 127 71.44) (width 0.25) (layer F.Cu) (net 9))
+  (zone (net 2) (net_name GND) (layer F.Cu) (hatch edge 0.508)
+    (connect_pads (clearance 0.254))
+    (min_thickness 0.254)
+    (fill yes (arc_segments 16) (thermal_gap 0.508) (thermal_bridge_width 0.508))
+    (polygon
+      (pts
+        (xy 116.85 65.95) (xy 116.85 74.3) (xy 140.35 74.3) (xy 140.35 65.95)
+      )
+    )
+  )
+  (zone (net 2) (net_name GND) (layer B.Cu) (hatch edge 0.508)
+    (connect_pads (clearance 0.254))
+    (min_thickness 0.254)
+    (fill yes (arc_segments 16) (thermal_gap 0.508) (thermal_bridge_width 0.508))
+    (polygon
+      (pts
+        (xy 116.85 65.95) (xy 116.85 74.3) (xy 140.35 74.3) (xy 140.35 65.95)
+      )
+    )
+  )
 )
